Commit message: Making arm_simple.urdf to have link lengths of 10, 20 and 20 cm

File: urdf/arm_simple.urdf (robot description, URDF)
Before this commit: robot visual, 6 links, 5 joints
Links:
- removed link link4
- added link tip; visual box size=0.04 0.015 0.025
- link base_link: geometry visual cylinder length=0.01 radius=0.05
- link link1: geometry visual cylinder length=0.1 radius=0.02
- link link2: geometry visual box size=0.2 0.01 0.02
- link link3: geometry visual box size=0.2 0.01 0.02
Joints:
- removed joint base_to_link1
- removed joint link1_to_link2
- removed joint link2_to_link3
- removed joint link3_to_link4
- added joint arti1: type revolute, parent link1, child link2, origin xyz=0.0 0.0 0.1 rpy=0 0 0, axis 0 1 0, limit lower=-1.58 upper=0.22 effort=1000.0 velocity=0.5
- added joint arti2: type revolute, parent link2, child link3, origin xyz=0.2 0.0 0.0 rpy=0 0 0, axis 0 1 0, limit lower=-1.58 upper=1.58 effort=1000.0 velocity=0.5
- added joint base: type revolute, parent base_link, child link1, origin xyz=0.0 0.0 0.0 rpy=0 0 0, axis 0 0 1, limit lower=-1.507 upper=1.507 effort=1000.0 velocity=0.5
- added joint tip: type fixed, parent link3, child tip, origin xyz=0.2 0 0 rpy=0 0 0, axis 0 0 1
- joint world_to_base: origin xyz=0 0 0 rpy=0 0 0 -> xyz=0.15 0.15 0 rpy=0 0 0
